Commit message: xacro is finished, gazebo launch files is created

File: urdf/links_joints.xacro (robot description, xacro)
@@ -11,5 +11,5 @@
         <color rgba="1 1 1 1"/>
     </material>
-<!-- *************************************colors********************************************-->
+<!-- *************************************functions ********************************************-->
   <xacro:macro name="m_joint" params="name type axis_xyz origin_rpy origin_xyz parent child limit_e limit_l limit_u limit_v">
     <joint name="${name}" type="${type}">
@@ -21,17 +21,5 @@
     </joint>
   </xacro:macro>
-  <xacro:macro name="m_link_cylinder" params="name origin_xyz origin_rpy radius length color">
-    <link name="${name}">
-        <origin rpy="${origin_rpy}" xyz="${origin_xyz}"/>
-      <visual>
-        <origin rpy="${origin_rpy}" xyz="${origin_xyz}"/>
-        <geometry>
-          <cylinder radius="${radius}" length="${length}"/>
-        </geometry>
-        <material name="${color}"/>
-      </visual>
-    </link>
-  </xacro:macro>
-  <xacro:macro name="m_link_box" params="name origin_xyz origin_rpy size mass ixx ixy ixz iyy iyz izz">
+  <xacro:macro name="m_link_cylinder" params="name origin_xyz origin_rpy radius length color mass ixx ixy ixz iyy iyz izz">
     <link name="${name}">
       <inertial>
@@ -43,5 +31,5 @@
         <origin rpy="${origin_rpy}" xyz="${origin_xyz}" />
         <geometry>
-          <box size="${size}" />
+          <cylinder radius="${radius}" length="${length}" />
         </geometry>
       </collision>
@@ -49,5 +37,6 @@
         <origin rpy="${origin_rpy}" xyz="${origin_xyz}" />
         <geometry>
-          <box size="${size}" />
+          <cylinder radius="${radius}" length="${length}" />
+          <material name="${color}"/>
         </geometry>
       </visual>

File: urdf/manipulator.xacro (robot description, xacro)
@@ -10,4 +10,8 @@
         origin_xyz="0 0 0"
         radius="0.08" length="0.03"
+        mass= "102"
+        ixx ="17.667" ixy ="17.667" ixz="0"
+        iyy ="17.667" iyz="0"
+        izz ="17.667"
         color="black"/>
     <m_joint name="${l000}__${l00}"
@@ -22,4 +26,8 @@
         origin_xyz="0 0 0.015"
         length="0.05" radius="0.06"
+        mass= "102"
+        ixx ="17.667" ixy ="17.667" ixz="0"
+        iyy ="17.667" iyz="0"
+        izz ="17.667"
         color="black"/>
     <m_joint name="${l00}__${l01}"
@@ -34,4 +42,8 @@
         origin_xyz="0 0 0.02"
         length="0.033" radius="0.03"
+        mass= "102"
+        ixx ="17.667" ixy ="17.667" ixz="0"
+        iyy ="17.667" iyz="0"
+        izz ="17.667"
         color="white"/>
     <m_joint name="${l01}__${l02}"
@@ -46,4 +58,8 @@
         origin_xyz="0 0 0.055"
         length="0.105" radius="0.03"
+        mass= "102"
+        ixx ="17.667" ixy ="17.667" ixz="0"
+        iyy ="17.667" iyz="0"
+        izz ="17.667"
         color="black"/>
     <m_joint name="${l02}__${l03}"
@@ -58,4 +74,8 @@
         origin_xyz="0 0 0.052"
         length="0.098" radius="0.03"
+        mass= "102"
+        ixx ="17.667" ixy ="17.667" ixz="0"
+        iyy ="17.667" iyz="0"
+        izz ="17.667"
         color="white"/>
     <m_joint name="${l03}__${l04}"
@@ -70,4 +90,8 @@
         origin_xyz="0 0 0.016"
         length="0.027" radius="0.03"
+        mass= "102"
+        ixx ="17.667" ixy ="17.667" ixz="0"
+        iyy ="17.667" iyz="0"
+        izz ="17.667"
         color="black"/>
     <m_joint name="${l04}__${l05}"
@@ -82,4 +106,8 @@
         origin_xyz="0 0 0.035"
         length="0.065" radius="0.03"
+        mass= "1.056"
+        ixx ="0.2667" ixy ="0" ixz="0"
+        iyy ="0.2667" iyz="0"
+        izz ="0.2667"
         color="white"/>
 <!-- *************************************link_01*********************************************-->

Commit message: gazebo simulation with 3 joints is working

File: urdf/links_joints.xacro (robot description, xacro)
@@ -20,6 +20,16 @@
       <child link="${child}" />
     </joint>
+    <transmission name="trans_${name}">
+      <type>transmission_interface/SimpleTransmission</type>
+      <joint name="${name}">
+        <hardwareInterface>hardware_interface/EffortJointInterface</hardwareInterface>
+      </joint>
+      <actuator name="motor_${name}">
+        <hardwareInterface>hardware_interface/EffortJointInterface</hardwareInterface>
+        <mechanicalReduction>1</mechanicalReduction>
+      </actuator>
+    </transmission>
   </xacro:macro>
-  <xacro:macro name="m_link_cylinder" params="name origin_xyz origin_rpy radius length color mass ixx ixy ixz iyy iyz izz">
+ <xacro:macro name="m_link_cylinder" params="name origin_xyz origin_rpy radius length color mass ixx ixy ixz iyy iyz izz">
     <link name="${name}">
       <inertial>
@@ -38,5 +48,5 @@
         <geometry>
           <cylinder radius="${radius}" length="${length}" />
-          <material name="${color}"/>
+          <material name="color"/>
         </geometry>
       </visual>

File: urdf/manipulator.xacro (robot description, xacro)
@@ -1,21 +1,22 @@
 <?xml version="1.0"?>
-<robot name="joy-it" xmlns:xacro="http://www.ros.org/wiki/xacro">
-    <!-- Include -->
-    <xacro:include filename="$(find robot_manipulator_5dof)/urdf/links_joints.xacro" />
-    <xacro:include filename="$(find robot_manipulator_5dof)/urdf/robot_parameters.xacro" />
-    <!-- Include -->
-<!-- *************************************bottom_link********************************************-->
+<robot name="joyit" xmlns:xacro="http://www.ros.org/wiki/xacro">
+    <xacro:include filename="$(find robot_manipulator_5dof)/urdf/links_joints.xacro"/>
+    <xacro:include filename="$(find robot_manipulator_5dof)/urdf/robot_parameters.xacro"/>
+    <!-- *************************************bottom_link********************************************-->
     <m_link_cylinder name="${l000}"
         origin_rpy="0 0 0"
         origin_xyz="0 0 0"
         radius="0.08" length="0.03"
-        mass= "102"
-        ixx ="17.667" ixy ="17.667" ixz="0"
-        iyy ="17.667" iyz="0"
-        izz ="17.667"
+        mass= "1024"
+        ixx ="1.0" ixy ="0.0" ixz="0.0"
+        iyy ="1.0" iyz="0.0"
+        izz ="1.0"
         color="black"/>
+    <gazebo reference="${l000}">
+        <material>Gazebo/Black</material>
+    </gazebo>
     <m_joint name="${l000}__${l00}"
-        type="fixed" axis_xyz="0 0 1"
-        limit_e="1000.0" limit_l="0" limit_u="3.14" limit_v="0.5"
+        type="revolute" axis_xyz="0 0 1"
+        limit_e="1000.0" limit_l="0.0" limit_u="0.0" limit_v="0.5"
         origin_rpy="0 0 0" origin_xyz="0 0 0.015"
         parent="${l000}"
@@ -26,9 +27,12 @@
         origin_xyz="0 0 0.015"
         length="0.05" radius="0.06"
-        mass= "102"
-        ixx ="17.667" ixy ="17.667" ixz="0"
-        iyy ="17.667" iyz="0"
-        izz ="17.667"
-        color="black"/>
+        mass= "1024"
+        ixx ="7.667" ixy ="7.667" ixz="0.0"
+        iyy ="7.667" iyz="0.0"
+        izz ="7.667"
+        color="white"/>
+    <gazebo reference="${l00}">
+        <material>Gazebo/Black</material>
+    </gazebo>
     <m_joint name="${l00}__${l01}"
         type="revolute" axis_xyz="0 0 1"
@@ -47,5 +51,8 @@
         izz ="17.667"
         color="white"/>
-    <m_joint name="${l01}__${l02}"
+    <gazebo reference="${l01}">
+        <material>Gazebo/White</material>
+    </gazebo>
+  <m_joint name="${l01}__${l02}"
         type="revolute" axis_xyz="0 1 0"
         limit_e="1000.0" limit_l="0" limit_u="3.14" limit_v="0.5"
@@ -62,53 +69,14 @@
         iyy ="17.667" iyz="0"
         izz ="17.667"
-        color="black"/>
-    <m_joint name="${l02}__${l03}"
-        type="revolute" axis_xyz="0 1 0"
-        limit_e="1000.0" limit_l="0" limit_u="3.14" limit_v="0.5"
-        origin_rpy="0 0 0" origin_xyz="0 0 0.105"
-        parent="${l02}"
-        child="${l03}"/>
-<!-- *************************************link_03*********************************************-->
-    <m_link_cylinder name="${l03}"
-        origin_rpy="0 0 0"
-        origin_xyz="0 0 0.052"
-        length="0.098" radius="0.03"
-        mass= "102"
-        ixx ="17.667" ixy ="17.667" ixz="0"
-        iyy ="17.667" iyz="0"
-        izz ="17.667"
         color="white"/>
-    <m_joint name="${l03}__${l04}"
-        type="revolute" axis_xyz="0 1 0"
-        limit_e="1000.0" limit_l="0" limit_u="3.14" limit_v="0.5"
-        origin_rpy="0 0 0" origin_xyz="0 0 0.098"
-        parent="${l03}"
-        child="${l04}"/>
-<!-- *************************************link_04*********************************************-->
-    <m_link_cylinder name="${l04}"
-        origin_rpy="0 0 0"
-        origin_xyz="0 0 0.016"
-        length="0.027" radius="0.03"
-        mass= "102"
-        ixx ="17.667" ixy ="17.667" ixz="0"
-        iyy ="17.667" iyz="0"
-        izz ="17.667"
-        color="black"/>
-    <m_joint name="${l04}__${l05}"
-        type="revolute" axis_xyz="0 0 1"
-        limit_e="1000.0" limit_l="0" limit_u="3.14" limit_v="0.5"
-        origin_rpy="0 0 0" origin_xyz="0 0 0.027"
-        parent="link_04"
-        child="link_05"/>
-<!-- *************************************link_05*********************************************-->
-    <m_link_cylinder name="${l05}"
-        origin_rpy="0 0 0"
-        origin_xyz="0 0 0.035"
-        length="0.065" radius="0.03"
-        mass= "1.056"
-        ixx ="0.2667" ixy ="0" ixz="0"
-        iyy ="0.2667" iyz="0"
-        izz ="0.2667"
-        color="white"/>
-<!-- *************************************link_01*********************************************-->
+<!-- ************************************* ROS control plugin ********************************-->
+<!-- To simulate model in order to pasrse the trasnmission tage and assign appropriate hardware interfaces
+ and the control manager -->
+    <gazebo>
+        <plugin name="gazebo_ros_control" filename="libgazebo_ros_control.so">
+            <robotNamespace>/joyit</robotNamespace>
+            <robotSimType>gazebo_ros_control/DefaultRobotHWSim</robotSimType>
+            <legacyModeNS>true</legacyModeNS>
+        </plugin>
+    </gazebo>
 </robot>

File: urdf/robot_parameters.xacro (robot description, xacro)
@@ -1,10 +1,10 @@
 <?xml version="1.0"?>
-<robot name="joy-it" xmlns:xacro="http://www.ros.org/wiki/xacro">
-    <xacro:property name="l000" value="bottom_link" />
-    <xacro:property name="l00" value="base_link" />
-    <xacro:property name="l01" value="link_01" />
-    <xacro:property name="l02" value="link_02" />
-    <xacro:property name="l03" value="link_03" />
-    <xacro:property name="l04" value="link_04" />
-    <xacro:property name="l05" value="link_05" />
+<robot name="joyit" xmlns:xacro="http://www.ros.org/wiki/xacro">
+    <xacro:property name="l000" value="bottom_link"/>
+    <xacro:property name="l00" value="base_link"/>
+    <xacro:property name="l01" value="link_01"/>
+    <xacro:property name="l02" value="link_02"/>
+    <xacro:property name="l03" value="link_03"/>
+    <xacro:property name="l04" value="link_04"/>
+    <xacro:property name="l05" value="link_05"/>
 </robot>

Commit message: whole robotic arm working in gazebo

File: urdf/links_joints.xacro (robot description, xacro)
@@ -1,4 +1,7 @@
 <?xml version="1.0" ?>
 <robot xmlns:xacro="http://www.ros.org/wiki/xacro">
+<!-- *************************************Constants*********************************** ******-->
+<xacro:property name="damping_value" value="50.0"/>
+<xacro:property name="friction_value" value="1.0"/>
 <!-- *************************************colors********************************************-->
     <material name="blue">
@@ -19,4 +22,5 @@
       <parent link="${parent}" />
       <child link="${child}" />
+      <dynamics damping="${damping_value}" friction="${friction_value}"/>
     </joint>
     <transmission name="trans_${name}">

File: urdf/manipulator.xacro (robot description, xacro)
@@ -4,22 +4,28 @@
     <xacro:include filename="$(find robot_manipulator_5dof)/urdf/robot_parameters.xacro"/>
     <!-- *************************************bottom_link********************************************-->
+    <link name="dummy_link">
+    </link>
+    <joint name="dummy_joint" type="fixed">
+        <parent link="dummy_link"/>
+        <child link="${l000}"/>
+    </joint>
     <m_link_cylinder name="${l000}"
         origin_rpy="0 0 0"
         origin_xyz="0 0 0"
         radius="0.08" length="0.03"
-        mass= "1024"
-        ixx ="1.0" ixy ="0.0" ixz="0.0"
-        iyy ="1.0" iyz="0.0"
-        izz ="1.0"
+        mass= "2000"
+        ixx ="0.0" ixy ="0.0" ixz="0.0"
+        iyy ="0.0" iyz="0.0"
+        izz ="0.0"
         color="black"/>
     <gazebo reference="${l000}">
         <material>Gazebo/Black</material>
     </gazebo>
-    <m_joint name="${l000}__${l00}"
-        type="revolute" axis_xyz="0 0 1"
-        limit_e="1000.0" limit_l="0.0" limit_u="0.0" limit_v="0.5"
-        origin_rpy="0 0 0" origin_xyz="0 0 0.015"
-        parent="${l000}"
-        child="${l00}"/>
+    <joint name="${l000}__${l00}" type="fixed">
+        <axis xyz="0 0 1"/>
+        <origin xyz="0 0 0.015" rpy="0 0 0"/>
+        <parent link="${l000}"/>
+        <child link="${l00}"/>
+    </joint>
 <!-- *************************************base_link*********************************************-->
     <m_link_cylinder name="${l00}"
@@ -27,8 +33,8 @@
         origin_xyz="0 0 0.015"
         length="0.05" radius="0.06"
-        mass= "1024"
-        ixx ="7.667" ixy ="7.667" ixz="0.0"
-        iyy ="7.667" iyz="0.0"
-        izz ="7.667"
+        mass= "2000"
+        ixx ="0.0" ixy ="0.0" ixz="0.0"
+        iyy ="0.0" iyz="0.0"
+        izz ="0.0"
         color="white"/>
     <gazebo reference="${l00}">
@@ -46,5 +52,5 @@
         origin_xyz="0 0 0.02"
         length="0.033" radius="0.03"
-        mass= "102"
+        mass= "1"
         ixx ="17.667" ixy ="17.667" ixz="0"
         iyy ="17.667" iyz="0"
@@ -56,5 +62,5 @@
   <m_joint name="${l01}__${l02}"
         type="revolute" axis_xyz="0 1 0"
-        limit_e="1000.0" limit_l="0" limit_u="3.14" limit_v="0.5"
+        limit_e="1000.0" limit_l="-3.14" limit_u="3.14" limit_v="0.5"
         origin_rpy="0 0 0" origin_xyz="0 0 0.033"
         parent="${l01}"
@@ -65,9 +71,70 @@
         origin_xyz="0 0 0.055"
         length="0.105" radius="0.03"
-        mass= "102"
+        mass= "1"
         ixx ="17.667" ixy ="17.667" ixz="0"
         iyy ="17.667" iyz="0"
         izz ="17.667"
         color="white"/>
+    <gazebo reference="${l02}">
+        <material>Gazebo/Grey</material>
+    </gazebo>
+    <m_joint name="${l02}__${l03}"
+        type="revolute" axis_xyz="0 1 0"
+        limit_e="1000.0" limit_l="0" limit_u="3.14" limit_v="0.5"
+        origin_rpy="0 0 0" origin_xyz="0 0 0.105"
+        parent="${l02}"
+        child="${l03}"/>
+<!-- *************************************link_03*********************************************-->
+    <m_link_cylinder name="${l03}"
+        origin_rpy="0 0 0"
+        origin_xyz="0 0 0.052"
+        length="0.098" radius="0.03"
+        mass= "1"
+        ixx ="17.667" ixy ="17.667" ixz="0"
+        iyy ="17.667" iyz="0"
+        izz ="17.667"
+        color="white"/>
+    <gazebo reference="${l03}">
+        <material>Gazebo/White</material>
+    </gazebo>
+    <m_joint name="${l03}__${l04}"
+        type="revolute" axis_xyz="0 1 0"
+        limit_e="1000.0" limit_l="0" limit_u="3.14" limit_v="0.5"
+        origin_rpy="0 0 0" origin_xyz="0 0 0.098"
+        parent="${l03}"
+        child="${l04}"/>
+<!-- *************************************link_04*********************************************-->
+    <m_link_cylinder name="${l04}"
+        origin_rpy="0 0 0"
+        origin_xyz="0 0 0.016"
+        length="0.027" radius="0.03"
+        mass= "1"
+        ixx ="17.667" ixy ="17.667" ixz="0"
+        iyy ="17.667" iyz="0"
+        izz ="17.667"
+        color="black"/>
+    <gazebo reference="${l04}">
+        <material>Gazebo/Grey</material>
+    </gazebo>
+    <m_joint name="${l04}__${l05}"
+        type="revolute" axis_xyz="0 0 1"
+        limit_e="1000.0" limit_l="0" limit_u="3.14" limit_v="0.5"
+        origin_rpy="0 0 0" origin_xyz="0 0 0.027"
+        parent="link_04"
+        child="link_05"/>
+<!-- *************************************link_05*********************************************-->
+    <m_link_cylinder name="${l05}"
+        origin_rpy="0 0 0"
+        origin_xyz="0 0 0.035"
+        length="0.065" radius="0.03"
+        mass= "1"
+        ixx ="0.2667" ixy ="0" ixz="0"
+        iyy ="0.2667" iyz="0"
+        izz ="0.2667"
+        color="white"/>
+    <gazebo reference="${l05}">
+        <material>Gazebo/White</material>
+    </gazebo>
+<!-- *************************************link_01*********************************************-->
 <!-- ************************************* ROS control plugin ********************************-->
 <!-- To simulate model in order to pasrse the trasnmission tage and assign appropriate hardware interfaces
